Commit message: Fixed missing link issue

File: models/youbot/youbot.urdf (robot description, URDF)
Before this commit: robot youbot, 21 links, 20 joints
Joints:
- joint youbot__arm_joint_0: type fixed -> revolute
- joint youbot__arm_joint_1: limit lower=0.0 upper=5.899213 effort=9.5 velocity=0.0 -> lower=0.0 upper=5.899213 effort=9.5 velocity=1.0
- joint youbot__arm_joint_2: limit lower=0.0 upper=2.70526 effort=9.5 velocity=-1.0 -> lower=0.0 upper=2.70526 effort=9.5 velocity=1.0
- joint youbot__arm_joint_3: limit lower=-5.183628 upper=0.0 effort=6.0 velocity=-1.0 -> lower=-5.183628 upper=0.0 effort=6.0 velocity=1.0
- joint youbot__arm_joint_4: limit lower=0.0 upper=3.577925 effort=2.0 velocity=-1.0 -> lower=0.0 upper=3.577925 effort=2.0 velocity=1.0
- joint youbot__arm_joint_5: limit lower=0.0 upper=5.846853 effort=1.0 velocity=-1.0 -> lower=0.0 upper=5.846853 effort=1.0 velocity=1.0
- joint youbot__base_footprint_joint: type fixed -> revolute
- joint youbot__base_laser_front_hokuyo_urg04_laser_joint: type fixed -> revolute
- joint youbot__caster_joint_bl: type fixed -> revolute
- joint youbot__caster_joint_br: type fixed -> revolute
- joint youbot__caster_joint_fl: type fixed -> revolute
- joint youbot__caster_joint_fr: type fixed -> revolute
- joint youbot__gripper_finger_joint_r: limit lower=0.0 upper=0.0115 effort=1.0 velocity=-1.0 -> lower=0.0 upper=0.0115 effort=1.0 velocity=1.0
- joint youbot__gripper_palm_joint: type fixed -> revolute
- joint youbot__plate_joint: type fixed -> revolute
- joint youbot__wheel_joint_bl: type fixed -> revolute
- joint youbot__wheel_joint_br: type fixed -> revolute
- joint youbot__wheel_joint_fl: type fixed -> revolute
- joint youbot__wheel_joint_fr: type fixed -> revolute
